File: peanut/pyro.kicad_sch (KiCad schematic)
At the start: 16 parts, among them J2 PYRO_OUT, Q2 NMOS, Q3 NMOS, Q4 NMOS

Commit message: feat: Verify component features
Completed most of the review checklist for the initial revision. Routing
can commence once design rules are updated.
Connections:
- net VBAT: no longer J2.1 (Pin_1), J2.3 (Pin_3)
- new net VBAT_RAW: J2.1 (Pin_1), J2.3 (Pin_3)
Other:
- note added: "4V2 -> 3V2 0V -> 0V"
- note added: "D"
- note added: "G"
- note added: "S"
- note added: "Vf = 2V If = 6.6mA - 2.42mA"
- note removed: "4V2 -> 3V3 0V -> 0V"
Changed lines of the file:
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@@
+		)
+	)
+	(text "D"
+		(exclude_from_sim no)
+		(at 47.752 107.188 0)
+		(effects
+			(font
+				(size 1.27 1.27)
+			)
 		)
 	)
@@
 		)
 	)
-	(text "4V2 -> 3V3\n0V -> 0V"
+	(text "Vf = 2V\nIf = 6.6mA - 2.42mA"
+		(exclude_from_sim no)
+		(at 69.342 88.646 0)
+		(effects
+			(font
+				(size 1.27 1.27)
+			)
+		)
+	)
+	(text "4V2 -> 3V2\n0V -> 0V"
 		(exclude_from_sim no)
 		(at 34.544 165.354 0)
@@
 		)
 	)
+	(text "G"
+		(exclude_from_sim no)
+		(at 44.704 114.554 0)
+		(effects
+			(font
+				(size 1.27 1.27)
+			)
+		)
+	)
 	(text "Continuity indicator LED (~5-10mA)"
 		(exclude_from_sim no)
 		(at 66.294 80.264 0)
+		(effects
+			(font
+				(size 1.27 1.27)
+			)
+		)
+	)
+	(text "S"
+		(exclude_from_sim no)
+		(at 48.26 119.38 0)
 		(effects
 			(font
@@
 		(dnp no)
 		(fields_autoplaced yes)
-		(property "Reference" "#PWR037"
+		(property "Reference" "#PWR058"
 			(at 196.85 93.98 0)
 			(hide yes)
@@
 			)
 		)
-		(property "Value" "VBAT"
+		(property "Value" "VBAT_RAW"
 			(at 196.85 85.09 0)
 			(show_name no)
@@
 			(project "peanut"
 				(path "/5c6b6cfc-6c84-425a-9b66-e6111713aae8/4be069cc-6620-4cc3-a173-eaa174b1ef03"
-					(reference "#PWR037")
+					(reference "#PWR058")
 					(unit 1)
 				)
@@
 	)
 	(symbol
+		(lib_id "power:VBUS")
+		(at 156.21 90.17 0)
+		(unit 1)
+		(body_style 1)
+		(exclude_from_sim no)
+		(in_bom yes)
+		(on_board yes)
+		(in_pos_files yes)
+		(dnp no)
+		(fields_autoplaced yes)
+		(property "Reference" "#PWR057"
+			(at 156.21 93.98 0)
+			(hide yes)
+			(show_name no)
+			(do_not_autoplace no)
+			(effects
+				(font
+					(size 1.27 1.27)
+				)
+			)
+		)
+		(property "Value" "VBAT_RAW"
+			(at 156.21 85.09 0)
+			(show_name no)
+			(do_not_autoplace no)
+			(effects
+				(font
+					(size 1.27 1.27)
+				)
+			)
+		)
+		(property "Footprint" ""
+			(at 156.21 90.17 0)
+			(hide yes)
+			(show_name no)
+			(do_not_autoplace no)
+			(effects
+				(font
+					(size 1.27 1.27)
+				)
+			)
+		)
+		(property "Datasheet" ""
+			(at 156.21 90.17 0)
+			(hide yes)
+			(show_name no)
+			(do_not_autoplace no)
+			(effects
+				(font
+					(size 1.27 1.27)
+				)
+			)
+		)
+		(property "Description" "Power symbol creates a global label with name \"VBUS\""
+			(at 156.21 90.17 0)
+			(hide yes)
+			(show_name no)
+			(do_not_autoplace no)
+			(effects
+				(font
+					(size 1.27 1.27)
+				)
+			)
+		)
+		(pin "1"
+		)
+		(instances
+			(project "peanut"
+				(path "/5c6b6cfc-6c84-425a-9b66-e6111713aae8/4be069cc-6620-4cc3-a173-eaa174b1ef03"
+					(reference "#PWR057")
+					(unit 1)
+				)
+			)
+		)
+	)
+	(symbol
 		(lib_id "Device:R")
 		(at 146.05 107.95 0)
@@
 					(unit 1)
 				)
-			)
-		)
-	)
-	(symbol
-		(lib_id "power:VBUS")
-		(at 156.21 90.17 0)
-		(unit 1)
-		(body_style 1)
-		(exclude_from_sim no)
-		(in_bom yes)
-		(on_board yes)
-		(in_pos_files yes)
-		(dnp no)
-		(fields_autoplaced yes)
-		(property "Reference" "#PWR035"
-			(at 156.21 93.98 0)
-			(hide yes)
-			(show_name no)
-			(do_not_autoplace no)
-			(effects
-				(font
-					(size 1.27 1.27)
-				)
-			)
-		)
-		(property "Value" "VBAT"
-			(at 156.21 85.09 0)
-			(show_name no)
-			(do_not_autoplace no)
-			(effects
-				(font
-					(size 1.27 1.27)
-				)
-			)
-		)
-		(property "Footprint" ""
-			(at 156.21 90.17 0)
-			(hide yes)
-			(show_name no)
-			(do_not_autoplace no)
-			(effects
-				(font
-					(size 1.27 1.27)
-				)
-			)
-		)
-		(property "Datasheet" ""
-			(at 156.21 90.17 0)
-			(hide yes)
-			(show_name no)
-			(do_not_autoplace no)
-			(effects
-				(font
-					(size 1.27 1.27)
-				)
-			)
-		)
-		(property "Description" "Power symbol creates a global label with name \"VBUS\""
-			(at 156.21 90.17 0)
-			(hide yes)
-			(show_name no)
-			(do_not_autoplace no)
-			(effects
-				(font
-					(size 1.27 1.27)
-				)
-			)
-		)
-		(pin "1"
-		)
-		(instances
-			(project "peanut"
-				(path "/5c6b6cfc-6c84-425a-9b66-e6111713aae8/4be069cc-6620-4cc3-a173-eaa174b1ef03"
-					(reference "#PWR035")
-					(unit 1)
-				)

Commit message: feat: Cheaper inductor
Swapped inductor for one that is cheaper. Current board cost (minus JST
connector since that is not available on Mouser) is $44.76 CAD in
components.
Parts:
- R10, R14, R18, R19: MPN SFR01MZPJ103 -> MCS04020C1002FE000
Changed lines of the file:
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@@
 			)
 		)
-		(property "MPN" "SFR01MZPJ103"
+		(property "MPN" "MCS04020C1002FE000"
 			(at 186.69 107.95 0)
 			(hide yes)
@@
 			)
 		)
-		(property "MPN" "SFR01MZPJ103"
+		(property "MPN" "MCS04020C1002FE000"
 			(at 83.82 142.24 90)
 			(hide yes)
@@
 			)
 		)
-		(property "MPN" "SFR01MZPJ103"
+		(property "MPN" "MCS04020C1002FE000"
 			(at 146.05 107.95 0)
 			(hide yes)
@@
 			)
 		)
-		(property "MPN" "SFR01MZPJ103"
+		(property "MPN" "MCS04020C1002FE000"
 			(at 46.99 142.24 90)
 			(hide yes)
