File: peanut/peanut.kicad_sch (KiCad schematic)
At the start: 41 parts, among them J1 USB-C, Q1 NMOS, U1 MS5611-01BA, U3 ESP32-C3FH4, Y1 40MHz +/-10ppm

Commit message: chore: re-annotate
Parts:
- renumbered C19 to C1, C9 to C10, C10 to C11, C11 to C12, C12 to C13, C13 to C14, C1 to C2, C2 to C3, C3 to C4, C4 to C5, C5 to C6, C6 to C7, C7 to C8, C8 to C9, D5 to D2, R26 to R10, R9 to R11, R7 to R5, R5 to R6, R6 to R7, R25 to R9
Changed lines of the file:
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@@
 		(dnp no)
 		(fields_autoplaced yes)
-		(property "Reference" "#PWR028"
+		(property "Reference" "#PWR030"
 			(at 237.49 53.34 0)
 			(hide yes)
@@
 			(project "peanut"
 				(path "/5c6b6cfc-6c84-425a-9b66-e6111713aae8"
-					(reference "#PWR028")
+					(reference "#PWR030")
 					(unit 1)
 				)
@@
 		(dnp no)
 		(fields_autoplaced yes)
-		(property "Reference" "#PWR025"
+		(property "Reference" "#PWR026"
 			(at 190.5 46.99 0)
 			(hide yes)
@@
 			(project "peanut"
 				(path "/5c6b6cfc-6c84-425a-9b66-e6111713aae8"
-					(reference "#PWR025")
+					(reference "#PWR026")
 					(unit 1)
 				)
@@
 		(dnp no)
 		(fields_autoplaced yes)
-		(property "Reference" "C11"
+		(property "Reference" "C12"
 			(at 194.31 35.5599 0)
 			(show_name no)
@@
 			(project "peanut"
 				(path "/5c6b6cfc-6c84-425a-9b66-e6111713aae8"
-					(reference "C11")
+					(reference "C12")
 					(unit 1)
 				)
@@
 		(dnp no)
 		(fields_autoplaced yes)
-		(property "Reference" "#PWR027"
+		(property "Reference" "#PWR029"
 			(at 232.41 99.06 0)
 			(hide yes)
@@
 			(project "peanut"
 				(path "/5c6b6cfc-6c84-425a-9b66-e6111713aae8"
-					(reference "#PWR027")
+					(reference "#PWR029")
 					(unit 1)
 				)
@@
 		(dnp no)
 		(fields_autoplaced yes)
-		(property "Reference" "#PWR02"
+		(property "Reference" "#PWR03"
 			(at 27.94 95.25 0)
 			(hide yes)
@@
 			(project "peanut"
 				(path "/5c6b6cfc-6c84-425a-9b66-e6111713aae8"
-					(reference "#PWR02")
+					(reference "#PWR03")
 					(unit 1)
 				)
@@
 		(dnp no)
 		(fields_autoplaced yes)
-		(property "Reference" "D5"
+		(property "Reference" "D2"
 			(at 228.6 75.8824 90)
 			(show_name no)
@@
 			(project "peanut"
 				(path "/5c6b6cfc-6c84-425a-9b66-e6111713aae8"
-					(reference "D5")
+					(reference "D2")
 					(unit 1)
 				)
@@
 		(dnp no)
 		(fields_autoplaced yes)
-		(property "Reference" "C6"
+		(property "Reference" "C7"
 			(at 124.46 35.5599 0)
 			(show_name no)
@@
 			(project "peanut"
 				(path "/5c6b6cfc-6c84-425a-9b66-e6111713aae8"
-					(reference "C6")
+					(reference "C7")
 					(unit 1)
 				)
@@
 		(dnp no)
 		(fields_autoplaced yes)
-		(property "Reference" "#PWR055"
+		(property "Reference" "#PWR024"
 			(at 184.15 110.49 0)
 			(hide yes)
@@
 			(project "peanut"
 				(path "/5c6b6cfc-6c84-425a-9b66-e6111713aae8"
-					(reference "#PWR055")
+					(reference "#PWR024")
 					(unit 1)
 				)
@@
 		(dnp no)
 		(fields_autoplaced yes)
-		(property "Reference" "#PWR056"
+		(property "Reference" "#PWR027"
 			(at 193.04 110.49 0)
 			(hide yes)
@@
 			(project "peanut"
 				(path "/5c6b6cfc-6c84-425a-9b66-e6111713aae8"
-					(reference "#PWR056")
+					(reference "#PWR027")
 					(unit 1)
 				)
@@
 		(dnp no)
 		(fields_autoplaced yes)
-		(property "Reference" "R25"
+		(property "Reference" "R9"
 			(at 186.69 109.2199 0)
 			(show_name no)
@@
 			(project "peanut"
 				(path "/5c6b6cfc-6c84-425a-9b66-e6111713aae8"
-					(reference "R25")
+					(reference "R9")
 					(unit 1)
 				)
@@
 		(dnp no)
 		(fields_autoplaced yes)
-		(property "Reference" "C9"
+		(property "Reference" "C10"
 			(at 158.75 35.5599 0)
 			(show_name no)
@@
 			(project "peanut"
 				(path "/5c6b6cfc-6c84-425a-9b66-e6111713aae8"
-					(reference "C9")
+					(reference "C10")
 					(unit 1)
 				)
@@
 		(dnp no)
 		(fields_autoplaced yes)
-		(property "Reference" "C7"
+		(property "Reference" "C8"
 			(at 134.62 35.5599 0)
 			(show_name no)
@@
 			(project "peanut"
 				(path "/5c6b6cfc-6c84-425a-9b66-e6111713aae8"
-					(reference "C7")
+					(reference "C8")
 					(unit 1)
 				)
@@
 		(dnp no)
 		(fields_autoplaced yes)
-		(property "Reference" "C3"
+		(property "Reference" "C4"
 			(at 58.42 33.0199 0)
 			(show_name no)
@@
 			(project "peanut"
 				(path "/5c6b6cfc-6c84-425a-9b66-e6111713aae8"
-					(reference "C3")
+					(reference "C4")
 					(unit 1)
 				)
@@
 		(dnp no)
 		(fields_autoplaced yes)
-		(property "Reference" "C2"
+		(property "Reference" "C3"
 			(at 43.18 114.2999 0)
 			(show_name no)
@@
 			(project "peanut"
 				(path "/5c6b6cfc-6c84-425a-9b66-e6111713aae8"
-					(reference "C2")
+					(reference "C3")
 					(unit 1)
 				)
@@
 		(dnp no)
 		(fields_autoplaced yes)
-		(property "Reference" "#FLG04"
+		(property "Reference" "#FLG01"
 			(at 45.72 145.415 0)
 			(hide yes)
@@
 			(project "peanut"
 				(path "/5c6b6cfc-6c84-425a-9b66-e6111713aae8"
-					(reference "#FLG04")
+					(reference "#FLG01")
 					(unit 1)
 				)
@@
 		(dnp no)
 		(fields_autoplaced yes)
-		(property "Reference" "C4"
+		(property "Reference" "C5"
 			(at 101.6 35.5599 0)
 			(show_name no)
@@
 			(project "peanut"
 				(path "/5c6b6cfc-6c84-425a-9b66-e6111713aae8"
-					(reference "C4")
+					(reference "C5")
 					(unit 1)
 				)
@@
 		(in_pos_files yes)
 		(dnp no)
-		(property "Reference" "C1"
+		(property "Reference" "C2"
 			(at 20.32 114.554 0)
 			(show_name no)
@@
 			(project "peanut"
 				(path "/5c6b6cfc-6c84-425a-9b66-e6111713aae8"
-					(reference "C1")
+					(reference "C2")
 					(unit 1)
 				)
@@
 		(in_pos_files yes)
 		(dnp no)
-		(property "Reference" "R6"
+		(property "Reference" "R7"
 			(at 74.93 182.88 90)
 			(show_name no)
@@
 			(project "peanut"
 				(path "/5c6b6cfc-6c84-425a-9b66-e6111713aae8"
-					(reference "R6")
+					(reference "R7")
 					(unit 1)
 				)
@@
 		(dnp no)
 		(fields_autoplaced yes)
-		(property "Reference" "#PWR026"
+		(property "Reference" "#PWR028"
 			(at 232.41 73.66 0)
 			(hide yes)
@@
 			(project "peanut"
 				(path "/5c6b6cfc-6c84-425a-9b66-e6111713aae8"
-					(reference "#PWR026")
+					(reference "#PWR028")
 					(unit 1)
 				)
@@
 		(dnp no)
 		(fields_autoplaced yes)
-		(property "Reference" "C12"
+		(property "Reference" "C13"
 			(at 234.95 40.6399 0)
 			(show_name no)
@@
 			(project "peanut"
 				(path "/5c6b6cfc-6c84-425a-9b66-e6111713aae8"
-					(reference "C12")
+					(reference "C13")
 					(unit 1)
 				)
@@
 		(dnp no)
 		(fields_autoplaced yes)
-		(property "Reference" "C10"
+		(property "Reference" "C11"
 			(at 184.15 35.5599 0)
 			(show_name no)
@@
 			(project "peanut"
 				(path "/5c6b6cfc-6c84-425a-9b66-e6111713aae8"
-					(reference "C10")
+					(reference "C11")
 					(unit 1)
 				)
@@
 		(dnp no)
 		(fields_autoplaced yes)
-		(property "Reference" "#PWR03"
+		(property "Reference" "#PWR01"
 			(at 26.67 191.77 0)
 			(hide yes)
@@
 			(project "peanut"
 				(path "/5c6b6cfc-6c84-425a-9b66-e6111713aae8"
-					(reference "#PWR03")
+					(reference "#PWR01")
 					(unit 1)
 				)
@@
 		(dnp no)
 		(fields_autoplaced yes)
-		(property "Reference" "#PWR024"
+		(property "Reference" "#PWR025"
 			(at 190.5 36.83 0)
 			(hide yes)
@@
 			(project "peanut"
 				(path "/5c6b6cfc-6c84-425a-9b66-e6111713aae8"
-					(reference "#PWR024")
+					(reference "#PWR025")
 					(unit 1)
 				)
@@
 		(dnp no)
 		(fields_autoplaced yes)
-		(property "Reference" "R7"
+		(property "Reference" "R5"
 			(at 72.39 80.0099 0)
 			(show_name no)
@@
 			(project "peanut"
 				(path "/5c6b6cfc-6c84-425a-9b66-e6111713aae8"
-					(reference "R7")
+					(reference "R5")
 					(unit 1)
 				)
@@
 		(dnp no)
 		(fields_autoplaced yes)
-		(property "Reference" "C13"
+		(property "Reference" "C14"
 			(at 247.65 40.6399 0)
 			(show_name no)
@@
 			(project "peanut"
 				(path "/5c6b6cfc-6c84-425a-9b66-e6111713aae8"
-					(reference "C13")
+					(reference "C14")
 					(unit 1)
 				)
@@
 		(in_pos_files yes)
 		(dnp no)
-		(property "Reference" "R5"
+		(property "Reference" "R6"
 			(at 74.93 172.72 90)
 			(show_name no)
@@
 			(project "peanut"
 				(path "/5c6b6cfc-6c84-425a-9b66-e6111713aae8"
-					(reference "R5")
+					(reference "R6")
 					(unit 1)
 				)
@@
 		(in_pos_files yes)
 		(dnp no)
-		(property "Reference" "C5"
+		(property "Reference" "C6"
 			(at 110.49 35.5599 0)
 			(show_name no)
@@
 			(project "peanut"
 				(path "/5c6b6cfc-6c84-425a-9b66-e6111713aae8"
-					(reference "C5")
+					(reference "C6")
 					(unit 1)
 				)
@@
 		(dnp no)
 		(fields_autoplaced yes)
-		(property "Reference" "C8"
+		(property "Reference" "C9"
 			(at 144.78 35.5599 0)
 			(show_name no)
@@
 			(project "peanut"
 				(path "/5c6b6cfc-6c84-425a-9b66-e6111713aae8"
-					(reference "C8")
+					(reference "C9")
 					(unit 1)
 				)
@@
 		(dnp no)
 		(fields_autoplaced yes)
-		(property "Reference" "R26"
+		(property "Reference" "R10"
 			(at 195.58 109.2199 0)
 			(show_name no)
@@
 			(project "peanut"
 				(path "/5c6b6cfc-6c84-425a-9b66-e6111713aae8"
-					(reference "R26")
+					(reference "R10")
 					(unit 1)
 				)
@@
 		(dnp no)
 		(fields_autoplaced yes)
-		(property "Reference" "R9"
+		(property "Reference" "R11"
 			(at 224.79 87.6299 0)
 			(show_name no)
@@
 			(project "peanut"
 				(path "/5c6b6cfc-6c84-425a-9b66-e6111713aae8"
-					(reference "R9")
+					(reference "R11")
 					(unit 1)
 				)
@@
 		(dnp no)
 		(fields_autoplaced yes)
-		(property "Reference" "C19"
+		(property "Reference" "C1"
 			(at 22.86 82.5499 0)
 			(show_name no)
@@
 			(project "peanut"
 				(path "/5c6b6cfc-6c84-425a-9b66-e6111713aae8"
-					(reference "C19")
+					(reference "C1")
 					(unit 1)
 				)
@@
 		(dnp no)
 		(fields_autoplaced yes)
-		(property "Reference" "#PWR01"
+		(property "Reference" "#PWR02"
 			(at 27.94 74.93 0)
 			(hide yes)
@@
 			(project "peanut"
 				(path "/5c6b6cfc-6c84-425a-9b66-e6111713aae8"
-					(reference "#PWR01")
+					(reference "#PWR02")
 					(unit 1)
 				)
